Commit message: Modified foot

File: src/robot_properties_solo/robot_properties_solo/xacro/leg.xacro (robot description, xacro)
@@ -368,5 +368,6 @@
         <origin xyz="0 0 0" rpy="0 0 0" />
         <geometry>
-          <mesh filename="package://robot_properties_solo/meshes/${mesh_ext}/with_foot/solo_foot.${mesh_ext}"/>
+          <sphere radius="0.02"/>
+          <!-- <mesh filename="package://robot_properties_solo/meshes/${mesh_ext}/with_foot/solo_foot.${mesh_ext}"/> -->
         </geometry>
         <material name="${color_name}">
@@ -378,5 +379,6 @@
         <origin xyz="0 0 0" rpy="0 0 0" />
         <geometry>
-            <mesh filename="package://robot_properties_solo/meshes/${mesh_ext}/with_foot/solo_foot.${mesh_ext}"/>
+          <sphere radius="0.02"/>
+            <!-- <mesh filename="package://robot_properties_solo/meshes/${mesh_ext}/with_foot/solo_foot.${mesh_ext}"/> -->
         </geometry>
         <material name="${color_name}">
